Commit message: Iris running with depth camera and ORBSLAM2

File: src/iris_description/gazebo/robot.gazebo.xacro (robot description, xacro)
@@ -1,212 +1,218 @@
 <?xml version="1.0"?>
 <robot xmlns:xacro="http://ros.org/wiki/xacro">
-    <!-- plugins -->
-    <!-- Lift Drag Plugins -->
-    <!-- <plugin name="rotor_0_blade_1" filename="libLiftDragPlugin.so">
-      <a0>0.3</a0>
-      <alpha_stall>1.4</alpha_stall>
-      <cla>4.2500</cla>
-      <cda>0.10</cda>
-      <cma>0.00</cma>
-      <cla_stall>-0.025</cla_stall>
-      <cda_stall>0.0</cda_stall>
-      <cma_stall>0.0</cma_stall>
-      <area>0.002</area>
-      <air_density>1.2041</air_density>
-      <cp>0.084 0 0</cp>
-      <forward>0 1 0</forward>
-      <upward>0 0 1</upward>
-      <link_name>$(arg namespace)/rotor_0</link_name>
-    </plugin>
-    <plugin name="rotor_0_blade_2" filename="libLiftDragPlugin.so">
-      <a0>0.3</a0>
-      <alpha_stall>1.4</alpha_stall>
-      <cla>4.2500</cla>
-      <cda>0.10</cda>
-      <cma>0.00</cma>
-      <cla_stall>-0.025</cla_stall>
-      <cda_stall>0.0</cda_stall>
-      <cma_stall>0.0</cma_stall>
-      <area>0.002</area>
-      <air_density>1.2041</air_density>
-      <cp>-0.084 0 0</cp>
-      <forward>0 -1 0</forward>
-      <upward>0 0 1</upward>
-      <link_name>$(arg namespace)/rotor_0</link_name>
-    </plugin>
-    <plugin name="rotor_1_blade_1" filename="libLiftDragPlugin.so">
-      <a0>0.3</a0>
-      <alpha_stall>1.4</alpha_stall>
-      <cla>4.2500</cla>
-      <cda>0.10</cda>
-      <cma>0.00</cma>
-      <cla_stall>-0.025</cla_stall>
-      <cda_stall>0.0</cda_stall>
-      <cma_stall>0.0</cma_stall>
-      <area>0.002</area>
-      <air_density>1.2041</air_density>
-      <cp>0.084 0 0</cp>
-      <forward>0 1 0</forward>
-      <upward>0 0 1</upward>
-      <link_name>$(arg namespace)/rotor_1</link_name>
-    </plugin>
-    <plugin name="rotor_1_blade_2" filename="libLiftDragPlugin.so">
-      <a0>0.3</a0>
-      <alpha_stall>1.4</alpha_stall>
-      <cla>4.2500</cla>
-      <cda>0.10</cda>
-      <cma>0.00</cma>
-      <cla_stall>-0.025</cla_stall>
-      <cda_stall>0.0</cda_stall>
-      <cma_stall>0.0</cma_stall>
-      <area>0.002</area>
-      <air_density>1.2041</air_density>
-      <cp>-0.084 0 0</cp>
-      <forward>0 -1 0</forward>
-      <upward>0 0 1</upward>
-      <link_name>$(arg namespace)/rotor_1</link_name>
-    </plugin>
-    <plugin name="rotor_2_blade_1" filename="libLiftDragPlugin.so">
-      <a0>0.3</a0>
-      <alpha_stall>1.4</alpha_stall>
-      <cla>4.2500</cla>
-      <cda>0.10</cda>
-      <cma>0.00</cma>
-      <cla_stall>-0.025</cla_stall>
-      <cda_stall>0.0</cda_stall>
-      <cma_stall>0.0</cma_stall>
-      <area>0.002</area>
-      <air_density>1.2041</air_density>
-      <cp>0.084 0 0</cp>
-      <forward>0 -1 0</forward>
-      <upward>0 0 1</upward>
-      <link_name>$(arg namespace)/rotor_2</link_name>
-    </plugin>
-    <plugin name="rotor_2_blade_2" filename="libLiftDragPlugin.so">
-      <a0>0.3</a0>
-      <alpha_stall>1.4</alpha_stall>
-      <cla>4.2500</cla>
-      <cda>0.10</cda>
-      <cma>0.00</cma>
-      <cla_stall>-0.025</cla_stall>
-      <cda_stall>0.0</cda_stall>
-      <cma_stall>0.0</cma_stall>
-      <area>0.002</area>
-      <air_density>1.2041</air_density>
-      <cp>-0.084 0 0</cp>
-      <forward>0 1 0</forward>
-      <upward>0 0 1</upward>
-      <link_name>$(arg namespace)/rotor_2</link_name>
-    </plugin>
-    <plugin name="rotor_3_blade_1" filename="libLiftDragPlugin.so">
-      <a0>0.3</a0>
-      <alpha_stall>1.4</alpha_stall>
-      <cla>4.2500</cla>
-      <cda>0.10</cda>
-      <cma>0.00</cma>
-      <cla_stall>-0.025</cla_stall>
-      <cda_stall>0.0</cda_stall>
-      <cma_stall>0.0</cma_stall>
-      <area>0.002</area>
-      <air_density>1.2041</air_density>
-      <cp>0.084 0 0</cp>
-      <forward>0 -1 0</forward>
-      <upward>0 0 1</upward>
-      <link_name>$(arg namespace)/rotor_3</link_name>
-    </plugin>
-    <plugin name="rotor_3_blade_2" filename="libLiftDragPlugin.so">
-      <a0>0.3</a0>
-      <alpha_stall>1.4</alpha_stall>
-      <cla>4.2500</cla>
-      <cda>0.10</cda>
-      <cma>0.00</cma>
-      <cla_stall>-0.025</cla_stall>
-      <cda_stall>0.0</cda_stall>
-      <cma_stall>0.0</cma_stall>
-      <area>0.002</area>
-      <air_density>1.2041</air_density>
-      <cp>-0.084 0 0</cp>
-      <forward>0 1 0</forward>
-      <upward>0 0 1</upward>
-      <link_name>$(arg namespace)/rotor_3</link_name>
-    </plugin> -->
-	<!-- ArduPilot Plugin -->
-  <xacro:macro name="ardupilot_macro" params="fdm_port">
-    <plugin name="arducopter_plugin" filename="libArduPilotPlugin.so">
-      <fdm_addr>127.0.0.1</fdm_addr>
-      <fdm_port_in>${fdm_port}</fdm_port_in>
-      <fdm_port_out>${fdm_port+1}</fdm_port_out>
-      <!--
-          Require by APM :
-          Only change model and gazebo from XYZ to XY-Z coordinates
-      -->
-      <modelXYZToAirplaneXForwardZDown>0 0 0 3.141593 0 0</modelXYZToAirplaneXForwardZDown>
-      <gazeboXYZToNED>0 0 0 3.141593 0 0</gazeboXYZToNED>
-      <imuName>$(arg namespace)/imu_link</imuName>
-      <connectionTimeoutMaxCount>5</connectionTimeoutMaxCount>
-      <control channel="0">
-      <!--
-          incoming control command [0, 1]
-          so offset it by 0 to get [0, 1]
-          and divide max target by 1.
-          offset = 0
-          multiplier = 838 max rpm / 1 = 838
-      -->
-      <type>VELOCITY</type>
-      <offset>0</offset>
-      <p_gain>0.20</p_gain>
-      <i_gain>0</i_gain>
-      <d_gain>0</d_gain>
-      <i_max>0</i_max>
-      <i_min>0</i_min>
-      <cmd_max>2.5</cmd_max>
-      <cmd_min>-2.5</cmd_min>
-      <jointName>$(arg namespace)/rotor_0_joint</jointName>
-      <multiplier>838</multiplier>
-      <controlVelocitySlowdownSim>1</controlVelocitySlowdownSim>
-      </control>
-      <control channel="1">
-      <type>VELOCITY</type>
-      <offset>0</offset>
-      <p_gain>0.20</p_gain>
-      <i_gain>0</i_gain>
-      <d_gain>0</d_gain>
-      <i_max>0</i_max>
-      <i_min>0</i_min>
-      <cmd_max>2.5</cmd_max>
-      <cmd_min>-2.5</cmd_min>
-      <jointName>$(arg namespace)/rotor_1_joint</jointName>
-      <multiplier>838</multiplier>
-      <controlVelocitySlowdownSim>1</controlVelocitySlowdownSim>
-      </control>
-      <control channel="2">
-      <type>VELOCITY</type>
-      <offset>0</offset>
-      <p_gain>0.20</p_gain>
-      <i_gain>0</i_gain>
-      <d_gain>0</d_gain>
-      <i_max>0</i_max>
-      <i_min>0</i_min>
-      <cmd_max>2.5</cmd_max>
-      <cmd_min>-2.5</cmd_min>
-      <jointName>$(arg namespace)/rotor_2_joint</jointName>
-      <multiplier>-838</multiplier>
-      <controlVelocitySlowdownSim>1</controlVelocitySlowdownSim>
-      </control>
-      <control channel="3">
-      <type>VELOCITY</type>
-      <offset>0</offset>
-      <p_gain>0.20</p_gain>
-      <i_gain>0</i_gain>
-      <d_gain>0</d_gain>
-      <i_max>0</i_max>
-      <i_min>0</i_min>
-      <cmd_max>2.5</cmd_max>
-      <cmd_min>-2.5</cmd_min>
-      <jointName>$(arg namespace)/rotor_3_joint</jointName>
-      <multiplier>-838</multiplier>
-      <controlVelocitySlowdownSim>1</controlVelocitySlowdownSim>
-      </control>
-    </plugin>
-  </xacro:macro>
+  <!-- plugins -->
+  <!-- Lift Drag Plugins -->
+  <!-- <gazebo reference="$(arg namespace)/rotor_0">
+      <plugin name="rotor_0_blade_1" filename="libLiftDragPlugin.so">
+        <a0>0.3</a0>
+        <alpha_stall>1.4</alpha_stall>
+        <cla>4.2500</cla>
+        <cda>0.10</cda>
+        <cma>0.00</cma>
+        <cla_stall>-0.025</cla_stall>
+        <cda_stall>0.0</cda_stall>
+        <cma_stall>0.0</cma_stall>
+        <area>0.002</area>
+        <air_density>1.2041</air_density>
+        <cp>0.084 0 0</cp>
+        <forward>0 1 0</forward>
+        <upward>0 0 1</upward>
+        <link_name>$(arg namespace)/rotor_0</link_name>
+      </plugin>
+      <plugin name="rotor_0_blade_2" filename="libLiftDragPlugin.so">
+        <a0>0.3</a0>
+        <alpha_stall>1.4</alpha_stall>
+        <cla>4.2500</cla>
+        <cda>0.10</cda>
+        <cma>0.00</cma>
+        <cla_stall>-0.025</cla_stall>
+        <cda_stall>0.0</cda_stall>
+        <cma_stall>0.0</cma_stall>
+        <area>0.002</area>
+        <air_density>1.2041</air_density>
+        <cp>-0.084 0 0</cp>
+        <forward>0 -1 0</forward>
+        <upward>0 0 1</upward>
+        <link_name>$(arg namespace)/rotor_0</link_name>
+      </plugin>
+  </gazebo>
+  <gazebo>
+      <plugin name="rotor_1_blade_1" filename="libLiftDragPlugin.so">
+        <a0>0.3</a0>
+        <alpha_stall>1.4</alpha_stall>
+        <cla>4.2500</cla>
+        <cda>0.10</cda>
+        <cma>0.00</cma>
+        <cla_stall>-0.025</cla_stall>
+        <cda_stall>0.0</cda_stall>
+        <cma_stall>0.0</cma_stall>
+        <area>0.002</area>
+        <air_density>1.2041</air_density>
+        <cp>0.084 0 0</cp>
+        <forward>0 1 0</forward>
+        <upward>0 0 1</upward>
+        <link_name>$(arg namespace)/rotor_1</link_name>
+      </plugin>
+      <plugin name="rotor_1_blade_2" filename="libLiftDragPlugin.so">
+        <a0>0.3</a0>
+        <alpha_stall>1.4</alpha_stall>
+        <cla>4.2500</cla>
+        <cda>0.10</cda>
+        <cma>0.00</cma>
+        <cla_stall>-0.025</cla_stall>
+        <cda_stall>0.0</cda_stall>
+        <cma_stall>0.0</cma_stall>
+        <area>0.002</area>
+        <air_density>1.2041</air_density>
+        <cp>-0.084 0 0</cp>
+        <forward>0 -1 0</forward>
+        <upward>0 0 1</upward>
+        <link_name>$(arg namespace)/rotor_1</link_name>
+      </plugin>
+      <plugin name="rotor_2_blade_1" filename="libLiftDragPlugin.so">
+        <a0>0.3</a0>
+        <alpha_stall>1.4</alpha_stall>
+        <cla>4.2500</cla>
+        <cda>0.10</cda>
+        <cma>0.00</cma>
+        <cla_stall>-0.025</cla_stall>
+        <cda_stall>0.0</cda_stall>
+        <cma_stall>0.0</cma_stall>
+        <area>0.002</area>
+        <air_density>1.2041</air_density>
+        <cp>0.084 0 0</cp>
+        <forward>0 -1 0</forward>
+        <upward>0 0 1</upward>
+        <link_name>$(arg namespace)/rotor_2</link_name>
+      </plugin>
+      <plugin name="rotor_2_blade_2" filename="libLiftDragPlugin.so">
+        <a0>0.3</a0>
+        <alpha_stall>1.4</alpha_stall>
+        <cla>4.2500</cla>
+        <cda>0.10</cda>
+        <cma>0.00</cma>
+        <cla_stall>-0.025</cla_stall>
+        <cda_stall>0.0</cda_stall>
+        <cma_stall>0.0</cma_stall>
+        <area>0.002</area>
+        <air_density>1.2041</air_density>
+        <cp>-0.084 0 0</cp>
+        <forward>0 1 0</forward>
+        <upward>0 0 1</upward>
+        <link_name>$(arg namespace)/rotor_2</link_name>
+      </plugin>
+      <plugin name="rotor_3_blade_1" filename="libLiftDragPlugin.so">
+        <a0>0.3</a0>
+        <alpha_stall>1.4</alpha_stall>
+        <cla>4.2500</cla>
+        <cda>0.10</cda>
+        <cma>0.00</cma>
+        <cla_stall>-0.025</cla_stall>
+        <cda_stall>0.0</cda_stall>
+        <cma_stall>0.0</cma_stall>
+        <area>0.002</area>
+        <air_density>1.2041</air_density>
+        <cp>0.084 0 0</cp>
+        <forward>0 -1 0</forward>
+        <upward>0 0 1</upward>
+        <link_name>$(arg namespace)/rotor_3</link_name>
+      </plugin>
+      <plugin name="rotor_3_blade_2" filename="libLiftDragPlugin.so">
+        <a0>0.3</a0>
+        <alpha_stall>1.4</alpha_stall>
+        <cla>4.2500</cla>
+        <cda>0.10</cda>
+        <cma>0.00</cma>
+        <cla_stall>-0.025</cla_stall>
+        <cda_stall>0.0</cda_stall>
+        <cma_stall>0.0</cma_stall>
+        <area>0.002</area>
+        <air_density>1.2041</air_density>
+        <cp>-0.084 0 0</cp>
+        <forward>0 1 0</forward>
+        <upward>0 0 1</upward>
+        <link_name>$(arg namespace)/rotor_3</link_name>
+      </plugin>
+    </gazebo> -->
+    <!-- ArduPilot Plugin -->
+    <xacro:macro name="ardupilot_macro" params="fdm_port">
+      <gazebo>
+        <plugin name="arducopter_plugin" filename="libArduPilotPlugin.so">
+          <fdm_addr>127.0.0.1</fdm_addr>
+          <fdm_port_in>${fdm_port}</fdm_port_in>
+          <fdm_port_out>${fdm_port+1}</fdm_port_out>
+          <!--
+              Require by APM :
+              Only change model and gazebo from XYZ to XY-Z coordinates
+          -->
+          <modelXYZToAirplaneXForwardZDown>0 0 0 3.141593 0 0</modelXYZToAirplaneXForwardZDown>
+          <gazeboXYZToNED>0 0 0 3.141593 0 0</gazeboXYZToNED>
+          <imuName>$(arg namespace)::$(arg namespace)/imu_link</imuName>
+          <connectionTimeoutMaxCount>5</connectionTimeoutMaxCount>
+          <control channel="0">
+          <!--
+              incoming control command [0, 1]
+              so offset it by 0 to get [0, 1]
+              and divide max target by 1.
+              offset = 0
+              multiplier = 838 max rpm / 1 = 838
+          -->
+          <type>VELOCITY</type>
+          <offset>0</offset>
+          <p_gain>0.20</p_gain>
+          <i_gain>0</i_gain>
+          <d_gain>0</d_gain>
+          <i_max>0</i_max>
+          <i_min>0</i_min>
+          <cmd_max>2.5</cmd_max>
+          <cmd_min>-2.5</cmd_min>
+          <jointName>$(arg namespace)::$(arg namespace)/rotor_0_joint</jointName>
+          <multiplier>838</multiplier>
+          <controlVelocitySlowdownSim>1</controlVelocitySlowdownSim>
+          </control>
+          <control channel="1">
+          <type>VELOCITY</type>
+          <offset>0</offset>
+          <p_gain>0.20</p_gain>
+          <i_gain>0</i_gain>
+          <d_gain>0</d_gain>
+          <i_max>0</i_max>
+          <i_min>0</i_min>
+          <cmd_max>2.5</cmd_max>
+          <cmd_min>-2.5</cmd_min>
+          <jointName>$(arg namespace)::$(arg namespace)/rotor_1_joint</jointName>
+          <multiplier>838</multiplier>
+          <controlVelocitySlowdownSim>1</controlVelocitySlowdownSim>
+          </control>
+          <control channel="2">
+          <type>VELOCITY</type>
+          <offset>0</offset>
+          <p_gain>0.20</p_gain>
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
File: src/iris_description/urdf/multirotor_base.xacro (robot description, xacro)
@@ -128,4 +128,38 @@
       </plugin>
     </gazebo>
+    <!-- <gazebo>
+      <plugin name="${robot_namespace}/rotor_${motor_number}_blade_1" filename="libLiftDragPlugin.so">
+        <a0>0.3</a0>
+        <alpha_stall>1.4</alpha_stall>
+        <cla>4.2500</cla>
+        <cda>0.10</cda>
+        <cma>0.00</cma>
+        <cla_stall>-0.025</cla_stall>
+        <cda_stall>0.0</cda_stall>
+        <cma_stall>0.0</cma_stall>
+        <area>0.002</area>
+        <air_density>1.2041</air_density>
+        <cp>0.084 0 0</cp>
+        <forward>0 1 0</forward>
+        <upward>0 0 1</upward>
+        <link_name>${robot_namespace}::${robot_namespace}/rotor_${motor_number}</link_name>
+      </plugin>
+      <plugin name="${robot_namespace}/rotor_${motor_number}_blade_2" filename="libLiftDragPlugin.so">
+        <a0>0.3</a0>
+        <alpha_stall>1.4</alpha_stall>
+        <cla>4.2500</cla>
+        <cda>0.10</cda>
+        <cma>0.00</cma>
+        <cla_stall>-0.025</cla_stall>
+        <cda_stall>0.0</cda_stall>
+        <cma_stall>0.0</cma_stall>
+        <area>0.002</area>
+        <air_density>1.2041</air_density>
+        <cp>-0.084 0 0</cp>
+        <forward>0 -1 0</forward>
+        <upward>0 0 1</upward>
+        <link_name>${robot_namespace}::${robot_namespace}/rotor_${motor_number}</link_name>
+      </plugin>
+    </gazebo> -->
     <gazebo reference="${robot_namespace}/rotor_${motor_number}">
       <material>Gazebo/${color}</material>
